File: LVDS-DP-Driver.kicad_sch (KiCad schematic)
At the start: 0 parts

Commit message: Signal Converting Part Done
Parts:
- added C (x6): C_Small, symbol Device:C_Small
- added J: 47272-0001, MOLEX_47272-0001, symbol 47272-0001:47272-0001
- added J: Conn_02x15_Odd_Even, symbol Connector_Generic:Conn_02x15_Odd_Even
- added R (x4): R_Small, symbol Device:R_Small
- added U (x3): CS5211, symbol Symbols:CS5211
Connections:
- new net: C.2, U.44 (AUXP)
- new net: J.14, R.1
- new net: C.2, U.62 (DP0N)
- new net: J.13, R.1
- new net: C.2, U.61 (DP0P)
- new net: C.2, U.65 (DP1N)
- new net: C.2, U.64 (DP1P)
- new net: C.2, U.43 (AUXN)
- new net A0N: J.7 (Pin_7), U.31 (LDC0N)
- new net A0P: J.8 (Pin_8), U.30 (LDC0P)
- new net A1N: J.9 (Pin_9), U.29 (LDC1N)
- new net A1P: J.10 (Pin_10), U.28 (LDC1P)
- new net A2N: J.11 (Pin_11), U.27 (LDC2N)
- new net A2P: J.12 (Pin_12), U.26 (LDC2P)
- new net A3N: J.17 (Pin_17), U.23 (LDC3N)
- new net A3P: J.18 (Pin_18), U.22 (LDC3P)
- new net ACLKN: J.15 (Pin_15), U.25 (LL1CN)
- new net ACLKP: J.16 (Pin_16), U.24 (LL1CP)
- new net B0N: J.19 (Pin_19), U.20 (LDC4N)
- new net B0P: J.20 (Pin_20), U.19 (LDC4P)
- new net B1N: J.21 (Pin_21), U.17 (LDC5N)
- new net B1P: J.22 (Pin_22), U.16 (LDC5P)
- new net B2N: J.23 (Pin_23), U.15 (LDC6N)
- new net B2P: J.24 (Pin_24), U.14 (LDC6P)
- new net B3N: J.29 (Pin_29), U.13 (LDC7N)
- new net B3P: J.30 (Pin_30), U.12 (LDC7P)
- new net BCLKN: J.27 (Pin_27), U.11 (LL2CN)
- new net BCLKP: J.28 (Pin_28), U.10 (LL2CP)
- new net DP_IN_HPD: R.2, U.59 (HPDET)
- new net GND: J.11, J.13 (Pin_13), J.14 (Pin_14), J.16, J.19, J.2, J.25 (Pin_25), J.26 (Pin_26), J.4 (Pin_4), J.5, J.5 (Pin_5), J.6 (Pin_6), J.8, J.S1 (SHIELD), J.S2 (SHIELD), J.S3 (SHIELD), J.S4 (SHIELD), R.1, R.2, R.2
- new net HPD_DET_DP0: J.18, R.1, R.2
- new net LCD_VCC: J.1 (Pin_1), J.2 (Pin_2), J.3 (Pin_3)
- new net RX_AUXN: C.1, J.17
- new net RX_AUXP: C.1, J.15
- new net RX_DP0N: C.1, J.10
- new net RX_DP0P: C.1, J.12
- new net RX_DP1N: C.1, J.7
- new net RX_DP1P: C.1, J.9
- no-connect marks 0 -> 5
