File: LVDS-DP-Driver.kicad_sch (KiCad schematic)
At the start: 151 parts, among them J1 47272-0001, J2 Conn_02x15_Odd_Even, J3 Conn_01x06_Male, J4 Conn_01x03_Male, J5 Conn_01x04_Male, J6 Conn_01x03_Male, Q1 AGM612AP, Q10 2N7002, Q11 AGM612AP, Q12 AGM308AP, Q13 AGM308AP, Q14 AGM308AP, Q15 AGM308AP, Q2 AGM612AP, Q3 AGM612AP, Q4 MMBT3904, Q5 MMBT3904, Q6 2N7002, Q7 AO3401A, Q8 2N7002, Q9 2N7002, U1 CS5211, U2 LM5176, U3 AT24C64, U5 LM25141, U8 LM25141, U9 TLV62130

Commit message: finish
Connections:
- net +3V3 is gone; now on net +3.3V: C54.1, J4.3 (Pin_3), Q10.1 (G), Q6.1 (G), R21.2, R22.1, R27.1, R28.1, R29.1, R30.1, R31.1, R37.1, R39.1, R40.1, R41.1, R42.1, R43.1, R44.1, R45.2, R46.2, U3.8 (VDD), U8.17 (VOUT)
Changed lines of the file:
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@@
+    )
+  )
+  (symbol (lib_name "+3V3_1") (lib_id "power:+3V3") (at 252.73 119.38 180) (unit 1)
+    (in_bom yes) (on_board yes) (dnp no) (fields_autoplaced)
+    (property "Reference" "#PWR0100" (at 252.73 115.57 0)
+      (effects (font (size 1.27 1.27)) hide)
+    )
+    (property "Value" "+3V3" (at 252.73 124.46 0)
+      (effects (font (size 1.27 1.27)))
+    )
+    (property "Footprint" "" (at 252.73 119.38 0)
+      (effects (font (size 1.27 1.27)) hide)
+    )
+    (property "Datasheet" "" (at 252.73 119.38 0)
+      (effects (font (size 1.27 1.27)) hide)
+    )
+    (pin "1")
+    (instances
+      (project "LVDS-DP-Driver"
+        (path "/46838880-46e6-40b4-8167-4d1ff56fb624"
+          (reference "#PWR0100") (unit 1)
+        )
+      )
     )
   )
@@
         )
       )
+    )
+  )
+  (symbol (lib_name "+3.3V_1") (lib_id "power:+3.3V") (at 252.73 119.38 0) (unit 1)
+    (in_bom yes) (on_board yes) (dnp no) (fields_autoplaced)
+    (property "Reference" "#PWR099" (at 252.73 123.19 0)
+      (effects (font (size 1.27 1.27)) hide)
+    )
+    (property "Value" "+3.3V" (at 252.73 114.3 0)
+      (effects (font (size 1.27 1.27)))
+    )
+    (property "Footprint" "" (at 252.73 119.38 0)
+      (effects (font (size 1.27 1.27)) hide)
+    )
+    (property "Datasheet" "" (at 252.73 119.38 0)
+      (effects (font (size 1.27 1.27)) hide)
+    )
+    (pin "1")
+    (instances
+      (project "LVDS-DP-Driver"
+        (path "/46838880-46e6-40b4-8167-4d1ff56fb624"
+          (reference "#PWR099") (unit 1)
+        )
+      )
