File: LVDS-DP-Driver.kicad_pcb (KiCad board)
At the start: 0 parts

Commit message: MOSFET and Inductors
Parts:
- added C1: 100nF, Capacitor_SMD:C_0603_1608Metric, F.Cu at (104.9, 29.0)
- added C10: 100nF, Capacitor_SMD:C_0603_1608Metric, F.Cu at (84.5, 45.3)
- added C11: 10pF, Capacitor_SMD:C_0603_1608Metric, F.Cu at (93.9, 36.5)
- added C12: 330uF, Capacitor_Tantalum_SMD:CP_EIA-7343-31_Kemet-D, F.Cu at (46.3, 44.1)
- added C13: 100nF, Capacitor_SMD:C_0603_1608Metric, F.Cu at (97.9, 31.5)
- added C14: 330uF, Capacitor_Tantalum_SMD:CP_EIA-7343-31_Kemet-D, F.Cu at (61.8, 30.6)
- added C15: 10pF, Capacitor_SMD:C_0603_1608Metric, F.Cu at (93.9, 31.5)
- added C16: 220pF, Capacitor_SMD:C_0603_1608Metric, F.Cu at (206.3, 39.6)
- added C17: 1.5nF, Capacitor_SMD:C_0603_1608Metric, F.Cu at (226.7, 23.3)
- added C18: 220pF, Capacitor_SMD:C_0603_1608Metric, F.Cu at (226.7, 18.2)
- added C19: 1.5nF, Capacitor_SMD:C_0603_1608Metric, F.Cu at (226.7, 20.8)
- added C2: 100nF, Capacitor_SMD:C_0603_1608Metric, F.Cu at (61.8, 68.8)
- added C20: 330pF, Capacitor_SMD:C_0603_1608Metric, F.Cu at (215.1, 36.0)
- added C21: 1.5nF, Capacitor_SMD:C_0603_1608Metric, F.Cu at (217.5, 27.1)
- added C22: 100nF, Capacitor_SMD:C_0603_1608Metric, F.Cu at (230.7, 18.2)
- added C23: 100nF, Capacitor_SMD:C_0603_1608Metric, F.Cu at (217.5, 29.6)
- added C24: 100nF, Capacitor_SMD:C_0603_1608Metric, F.Cu at (230.7, 20.8)
- added C25: 68nF, Capacitor_SMD:C_0603_1608Metric, F.Cu at (76.4, 44.4)
- added C26: 330uF, Capacitor_Tantalum_SMD:CP_EIA-7343-31_Kemet-D, F.Cu at (57.2, 42.9)
- added C27: 100nF, Capacitor_SMD:C_0603_1608Metric, F.Cu at (97.9, 36.5)
- added C28: 100nF, Capacitor_SMD:C_0603_1608Metric, F.Cu at (75.3, 56.9)
- added C29: 100nF, Capacitor_SMD:C_0603_1608Metric, F.Cu at (71.5, 46.3)
- added C3: 100nF, Capacitor_SMD:C_0603_1608Metric, F.Cu at (85.9, 34.8)
- added C30: 1uF, Capacitor_SMD:C_0603_1608Metric, F.Cu at (57.3, 61.5)
- added C31: 100nF, Capacitor_SMD:C_0603_1608Metric, F.Cu at (93.1, 39.1)
- added C32: 100nF, Capacitor_SMD:C_0603_1608Metric, F.Cu at (67.3, 57.4)
- added C33: 100nF, Capacitor_SMD:C_0603_1608Metric, F.Cu at (65.3, 59.9)
- added C34: 100nF, Capacitor_SMD:C_0603_1608Metric, F.Cu at (89.9, 31.5)
- added C35: 1uF, Capacitor_SMD:C_0603_1608Metric, F.Cu at (80.4, 42.8)
- added C36: 100nF, Capacitor_SMD:C_0603_1608Metric, F.Cu at (71.3, 56.3)
- added C37: 1uF, Capacitor_SMD:C_0603_1608Metric, F.Cu at (85.0, 40.3)
- added C38: 100nF, Capacitor_SMD:C_0603_1608Metric, F.Cu at (70.8, 51.3)
- added C39: 100nF, Capacitor_SMD:C_0603_1608Metric, F.Cu at (92.9, 29.0)
- added C4: 100nF, Capacitor_SMD:C_0603_1608Metric, F.Cu at (63.3, 57.4)
- added C40: 10uF, Capacitor_Tantalum_SMD:CP_EIA-3528-21_Kemet-B, F.Cu at (43.9, 67.7)
- added C42: 100nF, Capacitor_SMD:C_0603_1608Metric, F.Cu at (102.0, 34.0)
- added C43: 100nF, Capacitor_SMD:C_0603_1608Metric, F.Cu at (75.6, 46.9)
- added C44: 100nF, Capacitor_SMD:C_0603_1608Metric, F.Cu at (89.9, 36.6)
- added C45: 10uF, Capacitor_Tantalum_SMD:CP_EIA-3528-21_Kemet-B, F.Cu at (78.2, 29.9)
- added C5: 100nF, Capacitor_SMD:C_0603_1608Metric, F.Cu at (53.8, 68.4)
- added C6: 100nF, Capacitor_SMD:C_0603_1608Metric, F.Cu at (65.8, 62.4)
- added C7: 22uF, Capacitor_Tantalum_SMD:CP_EIA-3528-21_Kemet-B, F.Cu at (154.9, 17.5)
- added C8: 4.7uF, Capacitor_Tantalum_SMD:CP_EIA-3528-21_Kemet-B, F.Cu at (198.8, 43.5)
- added C9: 1nF, Capacitor_SMD:C_0603_1608Metric, F.Cu at (186.4, 45.0)
- added D1: D_Schottky, Diode_SMD:D_SOD-523, F.Cu at (210.1, 42.1)
- added D2: D_Schottky, Diode_SMD:D_SOD-523, F.Cu at (83.1, 52.8)
- added D3: D_Schottky, Diode_SMD:D_SOD-523, F.Cu at (69.6, 64.9)
- added D4: G, Diode_SMD:D_0603_1608Metric, F.Cu at (38.8, 56.0)
- added D5: O, Diode_SMD:D_0603_1608Metric, F.Cu at (88.9, 29.0)
- added J1: 47272-0001, Footprints:MOLEX_47272-0001, F.Cu at (136.6, 13.4)
- added J2: Conn_02x15_Odd_Even, Connector_PinHeader_2.00mm:PinHeader_2x15_P2.00mm_Vertical, F.Cu at (32.7, 29.7)
- added J3: Conn_01x06_Male, Connector_PinHeader_2.54mm:PinHeader_1x06_P2.54mm_Vertical, F.Cu at (39.1, 30.0)
- added J4: Conn_01x03_Male, Connector_PinHeader_2.54mm:PinHeader_1x03_P2.54mm_Vertical, F.Cu at (39.1, 47.4)
- added J5: Conn_01x04_Male, Connector_PinHeader_2.54mm:PinHeader_1x04_P2.54mm_Vertical, F.Cu at (54.6, 30.0)
- added J6: Conn_01x03_Male, Connector_PinHeader_2.54mm:PinHeader_1x03_P2.54mm_Vertical, F.Cu at (43.7, 49.3)
- added L1: 3.3uH, Inductor_SMD:L_TDK_NLV25_2.5x2.0mm, F.Cu at (173.4, 30.8)
- added L2: 3.3uH, Inductor_SMD:L_TDK_NLV25_2.5x2.0mm, F.Cu at (159.8, 17.3)
- added L3: 1.5uH, Inductor_SMD:L_1210_3225Metric, F.Cu at (162.8, 31.2)
- added Q1: Si4816BDY, Package_SO:SO-8_3.9x4.9mm_P1.27mm, F.Cu at (170.9, 26.0)
- added Q10: 2N7002, Package_TO_SOT_SMD:SOT-23, F.Cu at (59.3, 35.8)
- added Q2: Si4816BDY, Package_SO:SO-8_3.9x4.9mm_P1.27mm, F.Cu at (165.6, 18.5)
- added Q3: Si4816BDY, Package_SO:SO-8_3.9x4.9mm_P1.27mm, F.Cu at (168.1, 31.6)
- added Q4: MMBT3904, Package_TO_SOT_SMD:SOT-23, F.Cu at (52.8, 62.4)
- added Q5: MMBT3904, Package_TO_SOT_SMD:SOT-23, F.Cu at (66.4, 51.4)
- added Q6: 2N7002, Package_TO_SOT_SMD:SOT-23, F.Cu at (72.0, 42.8)
- added Q7: AO3401A, Package_TO_SOT_SMD:SOT-23, F.Cu at (49.4, 67.8)
- added Q8: 2N7002, Package_TO_SOT_SMD:SOT-23, F.Cu at (58.8, 57.8)
- added Q9: 2N7002, Package_TO_SOT_SMD:SOT-23, F.Cu at (81.5, 34.3)
- added R1: 1M, Resistor_SMD:R_0603_1608Metric, F.Cu at (210.3, 39.6)
- added R10: 20K, Resistor_SMD:R_0603_1608Metric, F.Cu at (84.5, 42.8)
- added R11: 4.75K, Resistor_SMD:R_0603_1608Metric, F.Cu at (93.1, 41.6)
- added R12: 1430, Resistor_SMD:R_1206_3216Metric, F.Cu at (84.0, 29.3)
- added R13: 105K, Resistor_SMD:R_0603_1608Metric, F.Cu at (100.9, 29.0)
- added R14: 20K, Resistor_SMD:R_0603_1608Metric, F.Cu at (75.3, 54.4)
- added R15: 15K, Resistor_SMD:R_0603_1608Metric, F.Cu at (221.5, 26.5)
- added R16: 18K, Resistor_SMD:R_0603_1608Metric, F.Cu at (225.5, 26.5)
- added R17: 10K, Resistor_SMD:R_0603_1608Metric, F.Cu at (215.1, 33.5)
- added R18: 2.43K, Resistor_SMD:R_0603_1608Metric, F.Cu at (69.3, 59.9)
- added R19: 1.82K, Resistor_SMD:R_0603_1608Metric, F.Cu at (80.4, 45.3)
- added R2: 1M, Resistor_SMD:R_0603_1608Metric, F.Cu at (203.8, 44.6)
- added R20: 25K, Resistor_SMD:R_0603_1608Metric, F.Cu at (61.8, 66.3)
- added R21: 20K, Resistor_SMD:R_0603_1608Metric, F.Cu at (89.0, 39.1)
- added R22: 1K, Resistor_SMD:R_0603_1608Metric, F.Cu at (96.9, 29.0)
- added R23: 1K, Resistor_SMD:R_0603_1608Metric, F.Cu at (71.5, 48.8)
- added R24: 10K, Resistor_SMD:R_0603_1608Metric, F.Cu at (83.6, 47.8)
- added R25: 1K, Resistor_SMD:R_0603_1608Metric, F.Cu at (89.0, 41.6)
- added R26: 10K, Resistor_SMD:R_0603_1608Metric, F.Cu at (65.8, 67.4)
- added R27: 1K, Resistor_SMD:R_0603_1608Metric, F.Cu at (63.3, 54.9)
- added R28: 10K, Resistor_SMD:R_0603_1608Metric, F.Cu at (57.8, 69.0)
- added R29: 10K, Resistor_SMD:R_0603_1608Metric, F.Cu at (67.3, 54.9)
- added R3: 1K, Resistor_SMD:R_0603_1608Metric, F.Cu at (73.3, 59.4)
- added R30: 10K, Resistor_SMD:R_0603_1608Metric, F.Cu at (57.8, 66.5)
- added R31: 10K, Resistor_SMD:R_0603_1608Metric, F.Cu at (53.8, 65.9)
- added R32: 4K7, Resistor_SMD:R_0603_1608Metric, F.Cu at (79.3, 55.3)
- added R33: 10K, Resistor_SMD:R_0603_1608Metric, F.Cu at (88.5, 46.6)
- added R34: 10K, Resistor_SMD:R_0603_1608Metric, F.Cu at (79.3, 52.8)
- added R35: 10K, Resistor_SMD:R_0603_1608Metric, F.Cu at (61.3, 61.2)
- added R36: 1K, Resistor_SMD:R_0603_1608Metric, F.Cu at (93.9, 34.0)
- added R37: 4K7, Resistor_SMD:R_0603_1608Metric, F.Cu at (85.9, 32.2)
- added R38: 4K7, Resistor_SMD:R_0603_1608Metric, F.Cu at (81.0, 40.3)
- added R39: 10K, Resistor_SMD:R_0603_1608Metric, F.Cu at (57.8, 64.0)
- added R4: 100K, Resistor_SMD:R_0603_1608Metric, F.Cu at (81.0, 37.8)
- added R40: 10K, Resistor_SMD:R_0603_1608Metric, F.Cu at (79.6, 50.3)
- added R41: 10K, Resistor_SMD:R_0603_1608Metric, F.Cu at (88.5, 44.1)
- added R42: 4K7, Resistor_SMD:R_0603_1608Metric, F.Cu at (76.4, 41.9)
- added R43: 4K7, Resistor_SMD:R_0603_1608Metric, F.Cu at (71.3, 53.8)
- added R44: 4K7, Resistor_SMD:R_0603_1608Metric, F.Cu at (97.9, 34.0)
- added R45: 4K7, Resistor_SMD:R_0603_1608Metric, F.Cu at (61.8, 63.8)
- added R46: 4K7, Resistor_SMD:R_0603_1608Metric, F.Cu at (69.9, 62.4)
- added R5: 10K, Resistor_SMD:R_0603_1608Metric, F.Cu at (182.4, 45.0)
- added R6: 3.16K, Resistor_SMD:R_0603_1608Metric, F.Cu at (206.3, 42.1)
- added R7: 4.75K, Resistor_SMD:R_0603_1608Metric, F.Cu at (221.5, 29.0)
- added R8: 1430, Resistor_SMD:R_1206_3216Metric, F.Cu at (58.3, 53.9)
- added R9: 63.4K, Resistor_SMD:R_0603_1608Metric, F.Cu at (89.9, 34.1)
- added SW1: SW_DIP_x04, Button_Switch_THT:SW_DIP_SPSTx04_Slide_6.7x11.72mm_W7.62mm_P2.54mm_LowProfile, F.Cu at (43.0, 30.6)
- added TP1: SMBUS_SDA, TestPoint:TestPoint_Pad_1.0x1.0mm, F.Cu at (96.6, 39.3)
- added TP2: SMBUS_SCL, TestPoint:TestPoint_Pad_1.0x1.0mm, F.Cu at (69.4, 67.6)
- added TP3: TestPoint, TestPoint:TestPoint_Pad_D4.0mm, F.Cu at (172.2, 18.3)
- added TP4: TestPoint, TestPoint:TestPoint_Pad_D4.0mm, F.Cu at (210.0, 35.3)
- added U1: CS5211, Package_DFN_QFN:QFN-68-1EP_8x8mm_P0.4mm_EP5.2x5.2mm, F.Cu at (35.8, 64.9)
- added U2: LTC3853, Package_DFN_QFN:QFN-40-1EP_6x6mm_P0.5mm_EP4.6x4.6mm, F.Cu at (163.4, 25.2)
- added U3: AT24C64, Package_SO:SOIC-8_3.9x4.9mm_P1.27mm, F.Cu at (71.0, 30.9)
Routing:
- net +12V: track 0.00 -> 51.5 mm, vias 0 -> 15
- net Net-(Q1-C): track 0.00 -> 19.8 mm
- net Net-(D1-A): track 0.00 -> 15.6 mm
- net Net-(Q2-C): track 0.00 -> 12.3 mm, vias 0 -> 4
- net /TG3: track 0.00 -> 10.5 mm, vias 0 -> 2
- net Net-(Q2-G2): track 0.00 -> 9.40 mm, vias 0 -> 2
- net Net-(Q1-G2): track 0.00 -> 7.53 mm, vias 0 -> 2
- net /BG3: track 0.00 -> 5.81 mm
- net Net-(Q2-G1): track 0.00 -> 4.17 mm, vias 0 -> 2
- net Net-(Q1-G1): track 0.00 -> 2.38 mm
- net GND: vias 0 -> 60
- added copper zone on F.Cu, net +12V
- added copper zone on F.Cu, net /SW3
- added copper zone on B.Cu, net GND
- added copper zone on F.Cu, net GND
- added copper zone on F.Cu, net Net-(Q1-C)
- added copper zone on F.Cu, net Net-(Q2-C)
Other:
- board outline added: 50 x 50 mm
- copper layers 0 -> 2
