File: LVDS-DP-Driver.kicad_pcb (KiCad board)
At the start: 2 copper layers, 152 parts, among them J1 47272-0001, J2 Conn_02x15_Odd_Even, J3 Conn_01x06_Male, J4 Conn_01x03_Male, J5 Conn_01x04_Male, J6 Conn_01x03_Male, Q1 AGM612AP, Q10 2N7002, Q11 AGM612AP, Q12 AGM308AP, Q13 AGM308AP, Q14 AGM308AP, Q15 AGM308AP, Q2 AGM612AP, Q3 AGM612AP, Q4 MMBT3904, Q5 MMBT3904, Q6 2N7002, Q7 AO3401A, Q8 2N7002, Q9 2N7002, U1 CS5211, U2 LM5176, U3 AT24C64, U5 LM25141, U8 LM25141, U9 TLV62130

Commit message: reconstruct
Parts:
- removed R15: 10K, Resistor_SMD:R_0603_1608Metric
- added REF**: Texas_DSBGA-5_0.822x1.116mm_Layout2x1x2_P0.4mm, Package_BGA:Texas_DSBGA-5_0.822x1.116mm_Layout2x1x2_P0.4mm, F.Cu at (79.8, 89.6)
- D1: value MBR180S1-7 -> MBR0580S1-7; footprint Diode_SMD:D_SMA -> Diode_SMD:D_SOD-123
- D2: value DSK12 -> B5817WS-MS; footprint Diode_SMD:D_SOD-123F -> Diode_SMD:D_SOD-323
- D3: value RB160MM-90TR -> B110WS; footprint Diode_SMD:D_SOD-123F -> Diode_SMD:D_SOD-323
- U5, U8: footprint Package_DFN_QFN:QFN-24-1EP_4x4mm_P0.5mm_EP2.15x2.15mm_ThermalVias -> Package_DFN_QFN:VQFN-24-1EP_4x4mm_P0.5mm_EP2.5x2.5mm_ThermalVias
- U9: footprint Package_DFN_QFN:VQFN-16-1EP_3x3mm_P0.5mm_EP1.1x1.1mm -> Package_DFN_QFN:VQFN-16-1EP_3x3mm_P0.5mm_EP1.6x1.6mm
- moved J2 140.3 mm to (58.7, 132.8), turned to -90 degrees
- moved U8 135.0 mm to (78.2, 132.3), turned to -90 degrees
- moved U5 129.8 mm to (79.7, 120.7), turned to 90 degrees
- moved C54 129.6 mm to (77.2, 138.9)
- moved U1 127.8 mm to (40.9, 119.9), turned to 45 degrees
- moved C56 123.4 mm to (74.9, 136.7), turned to 90 degrees
- moved R3 122.8 mm to (40.6, 111.0), turned to -90 degrees
- moved R54 121.3 mm to (77.2, 135.9)
- moved R4 120.1 mm to (30.2, 99.3), turned to -90 degrees
- moved C55 119.7 mm to (85.6, 133.6)
- moved R2 119.3 mm to (30.2, 93.2), turned to 90 degrees
- moved R21 119.2 mm to (77.2, 137.4), turned to 180 degrees
- moved C1 116.7 mm to (37.6, 111.0), turned to -90 degrees
- moved C57 116.3 mm to (85.6, 135.1)
- moved TP4 116.2 mm to (86.6, 138.9)
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Connections:
- net Net-(U1A-AUXN) renamed /AUXN
- net Net-(U1A-AUXP) renamed /AUXP
- net Net-(U1A-DP0N) renamed /DP0N
- net Net-(U1A-DP0P) renamed /DP0P
- net Net-(U1A-DP1N) renamed /DP1N
- net Net-(U1A-DP1P) renamed /DP1P
- J2 pad 1: /LCD_VCC -> HT
- J2 pad 2: /LCD_VCC -> HT
- J2 pad 3: /LCD_VCC -> HT
- J4 pad 3: +3.3V -> +3V3
- Q10 pad 1: +3.3V -> +3V3
- Q6 pad 1: +3.3V -> +3V3
- R22 pad 1: +3.3V -> +3V3
- R27 pad 1: +3.3V -> +3V3
- R28 pad 1: +3.3V -> +3V3
- R29 pad 1: +3.3V -> +3V3
- R30 pad 1: +3.3V -> +3V3
- R31 pad 1: +3.3V -> +3V3
- R37 pad 1: +3.3V -> +3V3
- R39 pad 1: +3.3V -> +3V3
- R40 pad 1: +3.3V -> +3V3
- R41 pad 1: +3.3V -> +3V3
- R42 pad 1: +3.3V -> +3V3
- R43 pad 1: +3.3V -> +3V3
- R44 pad 1: +3.3V -> +3V3
- R45 pad 2: +3.3V -> +3V3
- R46 pad 2: +3.3V -> +3V3
- TP3 pad 1: +12V -> VDC
- U2 pad 17: /MAIN_PG -> unconnected-(U2-PG-Pad17)
- U3 pad 8: +3.3V -> +3V3
- U8 pad 17: +5V -> +3V3
Routing:
- net GND: track 0.00 -> 57.1 mm, vias 0 -> 199
- net +12V: track 0.00 -> 33.3 mm, vias 0 -> 90
- net /HPD_DET_DP0: track 0.00 -> 25.7 mm, vias 0 -> 3
- net Net-(J1-Pad14): track 0.00 -> 22.4 mm
- net /SW1: track 0.00 -> 20.4 mm, vias 0 -> 68
- net /VCC: track 0.00 -> 20.3 mm, vias 0 -> 4
- net Net-(D6-K): track 0.00 -> 19.2 mm, vias 0 -> 2
- net Net-(J1-Pad13): track 0.00 -> 18.5 mm
- net /VINSNS: track 0.00 -> 17.9 mm, vias 0 -> 2
- net /A0N: track 0.00 -> 17.6 mm, vias 0 -> 1
- net /B3P: track 0.00 -> 17.5 mm
- net /A0P: track 0.00 -> 17.3 mm, vias 0 -> 1
- net /B3N: track 0.00 -> 17.3 mm
- net /ACLKN: track 0.00 -> 17.3 mm
- net /ACLKP: track 0.00 -> 17.0 mm
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- added copper zone on F.Cu, net +12V
- added copper zone on In2.Cu, net +12V
- added copper zone on In2.Cu, net +3.3V
- added copper zone on F.Cu, net +3V3
- added copper zone on F.Cu, net +5V
- added copper zone on In2.Cu, net +5V
- added copper zone on B.Cu, net /BUCK3_SW
- added copper zone on F.Cu, net /BUCK3_SW
- added copper zone on B.Cu, net /BUCK5_SW
- added copper zone on F.Cu, net /BUCK5_SW
- added copper zone on F.Cu, net /CS_3
- added copper zone on F.Cu, net /CS_5
- added copper zone on B.Cu, net /RCS
- added copper zone on F.Cu, net /RCS
- added copper zone on B.Cu, net /SW1
- added copper zone on F.Cu, net /SW1
- added copper zone on F.Cu, net /SW2
- added copper zone on F.Cu, net GND
- added copper zone on In1.Cu, net GND
- added copper zone on F.Cu, net Net-(U5-DEMB)
- added copper zone on F.Cu, net VDC
Other:
- board outline added: 60 x 50 mm
- copper layers 2 -> 4
- board text added: "0.1016 mm / 0.1016 mm"
- board text added: "0.3000 mm"
- board text added: "0.7901 mm"
- board text added: "4"
- board text added: "59.9900 mm x 50.0000 mm"
- board text added: "BOARD CHARACTERISTICS"
- board text added: "Board Thickness:"
- board text added: "Board overall dimensions:"
- board text added: "Castellated pads:"
- board text added: "Copper Finish:"
- board text added: "Copper Layer Count:"
- board text added: "Edge card connectors:"
- board text added: "Impedance Control:"
- board text added: "Min hole diameter:"
- board text added: "Min track/spacing:"
- board text added: "No"
- board text added: "None"
- board text added: "Plated Board Edge:"
- board text added: "Yes"

Commit message: file sync
Parts:
- moved L4 142.0 mm to (59.1, 120.9), turned to -90 degrees
- moved U9 137.7 mm to (61.6, 122.5)
- moved C62 137.6 mm to (65.5, 124.0), turned to 180 degrees
- moved C63 133.2 mm to (63.2, 118.6), turned to 90 degrees
- moved C64 132.4 mm to (61.7, 118.6), turned to 90 degrees
- moved R56 111.7 mm to (89.2, 119.5)
- moved R57 111.7 mm to (89.2, 122.0)
- moved R58 111.7 mm to (89.2, 124.5)
- moved C65 111.7 mm to (89.2, 117.0)
- moved C15 10.0 mm to (62.6, 111.8)
- moved C22 10.0 mm to (62.6, 116.3)
- moved C53 10.0 mm to (63.4, 136.7)
- moved R13 10.0 mm to (63.4, 114.0)
- moved R14 10.0 mm to (61.9, 114.0)
- moved C10 10.0 mm to (60.9, 106.4)
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Routing:
- net GND: track 57.1 -> 63.7 mm, vias 199 -> 202
- net Net-(U9-SS): track 0.00 -> 2.17 mm
- net +12V: vias 90 -> 99
- added copper zone on F.Cu, net Net-(L4-Pad1)
Other:
- board size 60 x 50 mm -> 50 x 50 mm
- board text added: "49.9900 mm x 50.0000 mm"
