File: LVDS-DP-Driver.kicad_pcb (KiCad board)
At the start: 4 copper layers, 50 x 50 mm, 152 parts, among them J1 47272-0001, J2 Conn_02x15_Odd_Even, J3 Conn_01x06_Male, J4 Conn_01x03_Male, J5 Conn_01x04_Male, J6 Conn_01x03_Male, Q1 AGM612AP, Q10 2N7002, Q11 AGM612AP, Q12 AGM308AP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

Commit message: finish
Parts:
- removed C42, C43, C44: 100nF, Capacitor_SMD:C_0603_1608Metric
- removed J5: Conn_01x04_Male, Connector_PinHeader_2.54mm:PinHeader_1x04_P2.54mm_Vertical
- removed R39, R40, R41, R56: 10K, Resistor_SMD:R_0603_1608Metric
- removed REF**: Texas_DSBGA-5_0.822x1.116mm_Layout2x1x2_P0.4mm, Package_BGA:Texas_DSBGA-5_0.822x1.116mm_Layout2x1x2_P0.4mm
- moved Q8 124.2 mm to (45.0, 138.9), turned to 90 degrees
- moved Q9 120.5 mm to (39.9, 138.9), turned to 90 degrees
- moved C34 115.2 mm to (63.2, 127.7), turned to -90 degrees
- moved R33 114.5 mm to (49.0, 138.7), turned to 90 degrees
- moved R34 111.9 mm to (47.5, 138.7), turned to -90 degrees
- moved C35 110.4 mm to (57.9, 127.0), turned to 180 degrees
- moved R29 109.6 mm to (49.8, 123.7), turned to -90 degrees
- moved Q7 109.6 mm to (51.6, 138.4), turned to 90 degrees
- moved C32 109.1 mm to (34.0, 123.2), turned to -45 degrees
- moved R35 109.1 mm to (42.4, 138.7), turned to -90 degrees
- moved R42 106.7 mm to (54.6, 120.7), turned to 90 degrees
- moved Q4 106.6 mm to (31.2, 119.6), turned to -90 degrees
- moved R36 106.6 mm to (37.3, 138.7), turned to -90 degrees
- moved R43 104.0 mm to (53.1, 120.7), turned to 90 degrees
- moved R31 103.2 mm to (48.3, 122.4), turned to 90 degrees
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Connections:
- C54 pad 1: +3V3 -> +3.3V
- J4 pad 3: +3V3 -> +3.3V
- Q10 pad 1: +3V3 -> +3.3V
- Q6 pad 1: +3V3 -> +3.3V
- R21 pad 2: +3V3 -> +3.3V
- R22 pad 1: +3V3 -> +3.3V
- R27 pad 1: +3V3 -> +3.3V
- R28 pad 1: +3V3 -> +3.3V
- R29 pad 1: +3V3 -> +3.3V
- R30 pad 1: +3V3 -> +3.3V
- R31 pad 1: +3V3 -> +3.3V
- R37 pad 1: +3V3 -> +3.3V
- R42 pad 1: +3V3 -> +3.3V
- R43 pad 1: +3V3 -> +3.3V
- R44 pad 1: +3V3 -> +3.3V
- R45 pad 2: +3V3 -> +3.3V
- R46 pad 2: +3V3 -> +3.3V
- U3 pad 8: +3V3 -> +3.3V
- U8 pad 17: +3V3 -> +3.3V
Routing:
- net +3.3V: track 0.00 -> 61.2 mm, vias 0 -> 35
- net /EN_VCC: track 0.00 -> 54.3 mm, vias 0 -> 2
- net HT: track 0.00 -> 47.5 mm, vias 0 -> 2
- net GND: track 63.7 -> 103.7 mm, vias 202 -> 266
- net +1V8: track 0.00 -> 38.3 mm, vias 0 -> 42
- net Net-(U1B-SSDA): track 0.00 -> 34.7 mm, vias 0 -> 2
- net Net-(U1B-SSCL): track 0.00 -> 32.5 mm, vias 0 -> 2
- net /PWM0: track 0.00 -> 23.1 mm, vias 0 -> 2
- net /E2_SDA: track 0.00 -> 18.0 mm, vias 0 -> 2
- net /EN_BKLT: track 0.00 -> 17.0 mm, vias 0 -> 2
- net Net-(Q8-D): track 0.00 -> 16.2 mm
- net /P_BKLT_EN: track 0.00 -> 15.2 mm
- net /E2_SCL: track 0.00 -> 15.0 mm, vias 0 -> 2
- net /GPIO3: track 0.00 -> 14.9 mm
- net /P_PWM: track 0.00 -> 14.4 mm, vias 0 -> 2
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- added copper zone on F.Cu, net +1V8
- added copper zone on In2.Cu, net +1V8
- added copper zone on B.Cu, net +3.3V
- added copper zone on F.Cu, net +3.3V
- added copper zone on B.Cu, net +5V
- added copper zone on F.Cu, net HT
- added copper zone on F.Cu, net Net-(J4-Pin_2)
- removed copper zone on F.Cu, net +3V3
