File: DP-Alternate-USB.kicad_sch (KiCad schematic)
At the start: 0 parts

Commit message: created subschem and C project
Parts:
- added C17: 1uF, Capacitor_SMD:C_0603_1608Metric, symbol OLED-rescue:C(MM)-LibCool
- added C41, C46: 220pF, symbol Device:C_Small
- added C47, C49, C50, C51: 100nF, symbol Device:C_Small
- added J7: USB_C_Receptacle, symbol Connector:USB_C_Receptacle
- added R47, R48, R49, R50, R51: 10K, symbol Device:R_Small
- added R52, R53: 2M, symbol Device:R_Small
- added U4: ~, symbol Symbols:TUSB422
- added U6: ~, symbol Symbols:TUSB564
- added U7: ~, symbol Symbols:STM32G030F6P6
Connections:
- new net: C17.1, U7.6 (NRST)
- new net: J7.A10 (RX2-), U6.15 (RX2n)
- new net: J7.A11 (RX2+), U6.16 (RX2p)
- new net: C49.1, J7.A2 (TX1+)
- new net: C47.1, J7.A3 (TX1-)
- new net: J7.B10 (RX1-), U6.13 (RX1n)
- new net: J7.B11 (RX1+), U6.12 (RX1p)
- new net: C51.1, J7.B2 (TX2+)
- new net: C50.1, J7.B3 (TX2-)
- new net: C51.2, U6.19 (TX2p)
- new net: C47.2, U6.10 (TX1n)
- new net: C50.2, U6.18 (TX2n)
- new net: C49.2, U6.9 (TX1p)
- new net +3.3V: R47.1, R48.1, R49.1, R50.2, R51.2, U7.4 (VDD)
- new net +3V3: U6.20 (VCC), U6.28 (VCC), U6.6 (VCC)
- new net 8M: U7.2 (PC14/PC9)
- new net CC1: C41.2, J7.A5 (CC1), U4.C1 (CC1)
- new net CC2: C46.2, J7.B5 (CC2), U4.A1 (CC2)
- new net CTL1: U6.23 (CTL1), U7.11 (PA4)
- new net EN: U6.29 (EN), U7.12 (PA5)
- new net GND: C17.2, C41.1, C46.1, J7.A1 (GND), J7.A12 (GND), J7.B1 (GND), J7.B12 (GND), J7.S1 (SHIELD), R52.2, R53.2, U4.C2 (GND), U6.41 (GND), U7.5 (GND)
- new net HPDIN: U6.32 (HPDIN), U7.13 (PA6)
- new net INT: R49.2, U4.B2 (INT_N), U7.15 (PB0/1/2/PA8)
- new net MCU_RX: U7.10 (PA3)
- new net MCU_TX: U7.9 (PA2)
- new net MUXSCL: R51.1, U6.21 (FLIP/SCL), U7.20 (PB3/4/5/6)
- new net MUXSDA: R50.1, U6.22 (CTL0/SDA), U7.1 (PB7/8)
- new net PDC_SCL: R47.2, U4.B3 (SCL), U7.17 (PA12)
- new net PDC_SDA: R48.2, U4.C3 (SDA), U7.16 (PA11)
- new net PDC_VDD: U4.A3 (VDD)
- new net RX_DP0N: U6.39 (DP0n)
- new net RX_DP0P: U6.40 (DP0p)
- new net RX_DP1N: U6.36 (DP1n)
- new net RX_DP1P: U6.37 (DP1p)
- new net SBU1: J7.A8 (SBU1), R52.1, U6.24 (SBU1)
- new net SBU2: J7.B8 (SBU2), R53.1, U6.25 (SBU2)
- new net SWCLK: U7.19 (PA14)
- new net SWDIO: U7.18 (PA13)
- new net VBUS: J7.A4 (VBUS), J7.A9 (VBUS), J7.B4 (VBUS), J7.B9 (VBUS), U4.A2 (VBUSIN)
- new net VCONN: U4.B1 (VCONN)
- no-connect marks 0 -> 9

Commit message: cleanup and reconstruct
Parts:
- removed C17: 1uF, Capacitor_SMD:C_0603_1608Metric, symbol OLED-rescue:C(MM)-LibCool
- removed C41, C46: 220pF, symbol Device:C_Small
- removed C47, C49, C50, C51: 100nF, symbol Device:C_Small
- removed J7: USB_C_Receptacle, symbol Connector:USB_C_Receptacle
- removed R47, R48, R49, R50, R51: 10K, symbol Device:R_Small
- removed R52, R53: 2M, symbol Device:R_Small
- removed U4: ~, symbol Symbols:TUSB422
- removed U6: ~, symbol Symbols:TUSB564
- removed U7: ~, symbol Symbols:STM32G030F6P6
Connections:
- no-connect marks 9 -> 0
